File: SolarBirdsongUnit/Hardware/Solar Birdsong PCB v1/SolarBirdsongShield_v1.sch (KiCad schematic (older format))
At the start: 12 parts

Commit message: Code updates
Solar birdsong unit - v13 now working
Update of poetry wall changes
Parts:
- removed C3: 100u, ~, symbol CP1
- removed C?: 100n, ~, symbol C
- removed SHIELD?: ARDUINO_SHIELD, FT:ARDUINO_SHIELD, symbol ARDUINO_SHIELD
- added C? (x2): 100nF, matts_components:C1_wide_lg_pad, symbol C
- added C?: 100uF, Capacitors_ThroughHole:C_Radial_D5_L6_P2.5, symbol CP1
- added C? (x2): 22pF, matts_components:C1_lg_pad, symbol C
- added D?: D_Schottky, REInnovationFootprint:TH_Diode_2, symbol D_Schottky
- added IC?: ATMEGA328P-P, matts_components:DIP-28__300_ELL, symbol ATMEGA328P-P
- added P?: CONN_01X06, symbol CONN_01X06
- added P?: ISP, symbol CONN_02X03
- added R?: 10k, REInnovationFootprint:TH_Resistor_1, symbol R
- added R?: 1k, ~, symbol R-RESCUE-SolarBirdsongShield_v1
- added SW?: RESET, matts_components:SW_PUSH_single_pins, symbol SPST
- added X?: 16MHz, matts_components:Xtal_small_matt, symbol CRYSTAL_16MHz
- C?: symbol C -> C-RESCUE-SolarBirdsongShield_v1
- R? (x4): symbol R -> R-RESCUE-SolarBirdsongShield_v1
Connections:
- net labels added: +5V, A0, A1, A2, A3, A4, A5, D10, D11, D12, D13, D2, D3, D4, D5, D6, D7, D8, D9, RESET, RxD, TxD, a0, a1, a2, a3, a4, a5, d0, d1, d10, d11, d12, d13, d2, d3, d4, d5, d6, d7, d8, d9
- wire segments 51 -> 118
- no-connect marks 0 -> 9
Other:
- note added: "1: RTS#\n2: Rx\n3: Tx\n4: Vcc\n5: CTS#\n6: GND"
- moved on the sheet: C?, K?, P?, Q?, R?, U?
