File: MovingWall/Hardware/StepperMotorController_12_v2/StepperMotorController_12_v2.sch (KiCad schematic (older format))
At the start: 26 parts, among them J1 ARDUINO_NANO_HEADER, K1 CONN_3, K2 CONN_3, K3 CONN_3, K4 CONN_3, P1 RESET_SW, P19 POWER_OUT, P2 SW1, P3 SW2, P4 POWER_IN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

Commit message: Updated with changes
Parts:
- C3: symbol CP1 -> CP1-RESCUE-StepperMotorController_12_v2
- D1, D3, D5, D7: symbol LED -> LED-RESCUE-StepperMotorController_12_v2
- R1, R2, R3, R4, R5, R7: symbol R -> R-RESCUE-StepperMotorController_12_v2
Changed lines of the file:
@@
 LIBS:contrib
 LIBS:valves
-LIBS:matts_components
-LIBS:uln-udn
-LIBS:arduino
-LIBS:w_connectors
 LIBS:StepperMotorController_12_v2-cache
 EELAYER 25 0
@@
 $EndSheet
 $Comp
-L R R3
+L R-RESCUE-StepperMotorController_12_v2 R3
 U 1 1 551B2385
 P 8150 3200
@@
 $EndComp
 $Comp
-L LED D3
+L LED-RESCUE-StepperMotorController_12_v2 D3
 U 1 1 551B23C1
 P 8150 2650
@@
 $EndComp
 $Comp
-L R R1
+L R-RESCUE-StepperMotorController_12_v2 R1
 U 1 1 551B24DC
 P 7950 3200
@@
 $EndComp
 $Comp
-L LED D1
+L LED-RESCUE-StepperMotorController_12_v2 D1
 U 1 1 551B24E2
 P 7950 2650
@@
 $EndComp
 $Comp
-L R R7
+L R-RESCUE-StepperMotorController_12_v2 R7
 U 1 1 551B2506
 P 8550 3200
@@
 $EndComp
 $Comp
-L LED D7
+L LED-RESCUE-StepperMotorController_12_v2 D7
 U 1 1 551B250C
 P 8550 2650
@@
 $EndComp
 $Comp
-L R R5
+L R-RESCUE-StepperMotorController_12_v2 R5
 U 1 1 551B2512
 P 8350 3200
@@
 $EndComp
 $Comp
-L LED D5
+L LED-RESCUE-StepperMotorController_12_v2 D5
 U 1 1 551B2518
 P 8350 2650
@@
 $EndComp
 $Comp
-L GND #PWR01
+L GND-RESCUE-StepperMotorController_12_v2 #PWR01
 U 1 1 551B255D
 P 8250 3600
@@
 $EndSheet
 $Comp
-L CP1 C3
+L CP1-RESCUE-StepperMotorController_12_v2 C3
 U 1 1 551B33BA
 P 6150 3200
@@
 $EndComp
 $Comp
-L GND #PWR02
+L GND-RESCUE-StepperMotorController_12_v2 #PWR02
 U 1 1 551B3CAB
 P 4300 2550
@@
 $EndComp
 $Comp
-L GND #PWR03
+L GND-RESCUE-StepperMotorController_12_v2 #PWR03
 U 1 1 551B457F
 P 5500 5650
@@
 $EndComp
 $Comp
-L GND #PWR06
+L GND-RESCUE-StepperMotorController_12_v2 #PWR06
 U 1 1 551D4012
 P 6400 3000
@@
 	4250 3400 4800 3400
 $Comp
-L GND #PWR08
+L GND-RESCUE-StepperMotorController_12_v2 #PWR08
 U 1 1 551EBD74
 P 2700 5200
@@
 NoConn ~ 4800 3200
 $Comp
-L GND #PWR09
+L GND-RESCUE-StepperMotorController_12_v2 #PWR09
 U 1 1 55A283C0
 P 4700 3300
@@
 	2500 2850 4250 2850
 $Comp
-L GND #PWR010
+L GND-RESCUE-StepperMotorController_12_v2 #PWR010
 U 1 1 55A2A5A7
 P 1800 3350
@@
 Connection ~ 2350 1800
 $Comp
-L R R4
+L R-RESCUE-StepperMotorController_12_v2 R4
 U 1 1 55CB5CF0
 P 2850 6750
@@
 $EndComp
 $Comp
-L R R2
+L R-RESCUE-StepperMotorController_12_v2 R2
 U 1 1 55CB6599
 P 2850 6000
@@
 $EndComp
 $Comp
-L GND #PWR012
+L GND-RESCUE-StepperMotorController_12_v2 #PWR012
 U 1 1 55CB6C0E
 P 2850 7150
